File: electronics/control_digital.kicad_sch (KiCad schematic)
At the start: 0 parts

Commit message: version en dos placas, pero con errores de tierra general. Se procede a versionar la PCB
Parts:
- added J10: MCP4725_fine_r2, Connector_PinSocket_2.54mm:PinSocket_1x06_P2.54mm_Vertical, symbol Connector:Conn_01x06_Socket
- added J11: MCP4725_coarse_r2, Connector_PinSocket_2.54mm:PinSocket_1x06_P2.54mm_Vertical, symbol Connector:Conn_01x06_Socket
- added J12: MCP4725_fine_r3, Connector_PinSocket_2.54mm:PinSocket_1x06_P2.54mm_Vertical, symbol Connector:Conn_01x06_Socket
- added J13: MCP4725_coarse_r3, Connector_PinSocket_2.54mm:PinSocket_1x06_P2.54mm_Vertical, symbol Connector:Conn_01x06_Socket
- added J14: MCP4725_fine_r4, Connector_PinSocket_2.54mm:PinSocket_1x06_P2.54mm_Vertical, symbol Connector:Conn_01x06_Socket
- added J15: MCP4725_coarse_r4, Connector_PinSocket_2.54mm:PinSocket_1x06_P2.54mm_Vertical, symbol Connector:Conn_01x06_Socket
- added J16: MCP4725_VBIAS, Connector_PinSocket_2.54mm:PinSocket_1x06_P2.54mm_Vertical, symbol Connector:Conn_01x06_Socket
- added J17: ADS1115, Connector_PinSocket_2.54mm:PinSocket_1x10_P2.54mm_Vertical, symbol Connector:Conn_01x10_Socket
- added J4, J5: Conn_01x19_Socket, Connector_PinSocket_2.54mm:PinSocket_1x19_P2.54mm_Vertical, symbol Connector:Conn_01x19_Socket
- added J6, J7: Conn_01x12_Socket, Connector_PinSocket_2.54mm:PinSocket_1x12_P2.54mm_Vertical, symbol Connector:Conn_01x12_Socket
- added J8: MCP4725_fine_r1, Connector_PinSocket_2.54mm:PinSocket_1x06_P2.54mm_Vertical, symbol Connector:Conn_01x06_Socket
- added J9: MCP4725_coarse_r1, Connector_PinSocket_2.54mm:PinSocket_1x06_P2.54mm_Vertical, symbol Connector:Conn_01x06_Socket
Connections:
- new net +3.3VDC: J10.5 (Pin_5), J11.5 (Pin_5), J12.5 (Pin_5), J13.5 (Pin_5), J14.5 (Pin_5), J15.5 (Pin_5), J16.5 (Pin_5), J17.1 (Pin_1), J4.1 (Pin_1), J6.1 (Pin_1), J8.5 (Pin_5), J9.5 (Pin_5)
- new net AGND_diff_pair: J17.8 (Pin_8)
- new net DGND: J10.2 (Pin_2), J10.6 (Pin_6), J11.2 (Pin_2), J11.6 (Pin_6), J12.2 (Pin_2), J12.6 (Pin_6), J13.2 (Pin_2), J13.6 (Pin_6), J14.2 (Pin_2), J14.6 (Pin_6), J15.2 (Pin_2), J15.6 (Pin_6), J16.2 (Pin_2), J16.6 (Pin_6), J17.2 (Pin_2), J4.14 (Pin_14), J5.13 (Pin_13), J5.19 (Pin_19), J6.2 (Pin_2), J8.2 (Pin_2), J8.6 (Pin_6), J9.2 (Pin_2), J9.6 (Pin_6)
- new net MCP_VBIAS_out: J16.1 (Pin_1)
- new net MCP_coarse_r1_out: J9.1 (Pin_1)
- new net MCP_coarse_r2_out: J11.1 (Pin_1)
- new net MCP_coarse_r3_out: J13.1 (Pin_1)
- new net MCP_coarse_r4_out: J15.1 (Pin_1)
- new net MCP_fine_r1_out: J8.1 (Pin_1)
- new net MCP_fine_r2_out: J10.1 (Pin_1)
- new net MCP_fine_r3_out: J12.1 (Pin_1)
- new net MCP_fine_r4_out: J14.1 (Pin_1)
- new net SCL_coarse_r1: J6.12 (Pin_12), J9.3 (Pin_3)
- new net SCL_coarse_r2: J11.3 (Pin_3), J7.4 (Pin_4)
- new net SCL_coarse_r3: J13.3 (Pin_3), J7.8 (Pin_8)
- new net SCL_coarse_r4: J15.3 (Pin_3), J7.12 (Pin_12)
- new net SCL_fine_r1: J6.10 (Pin_10), J8.3 (Pin_3)
- new net SCL_fine_r2: J10.3 (Pin_3), J7.2 (Pin_2)
- new net SCL_fine_r3: J12.3 (Pin_3), J7.6 (Pin_6)
- new net SCL_fine_r4: J14.3 (Pin_3), J7.10 (Pin_10)
- new net SCL_main: J16.3 (Pin_3), J17.4 (Pin_4), J5.17 (Pin_17), J6.4 (Pin_4)
- new net SDA_coarse_r1: J6.11 (Pin_11), J9.4 (Pin_4)
- new net SDA_coarse_r2: J11.4 (Pin_4), J7.3 (Pin_3)
- new net SDA_coarse_r3: J13.4 (Pin_4), J7.7 (Pin_7)
- new net SDA_coarse_r4: J15.4 (Pin_4), J7.11 (Pin_11)
- new net SDA_fine_r1: J6.9 (Pin_9), J8.4 (Pin_4)
- new net SDA_fine_r2: J10.4 (Pin_4), J7.1 (Pin_1)
- new net SDA_fine_r3: J12.4 (Pin_4), J7.5 (Pin_5)
- new net SDA_fine_r4: J14.4 (Pin_4), J7.9 (Pin_9)
- new net SDA_main: J16.4 (Pin_4), J17.3 (Pin_3), J5.15 (Pin_15), J6.3 (Pin_3)
- new net opto_1_out: J4.9 (Pin_9)
- new net opto_2_out: J4.10 (Pin_10)
- new net opto_3_out: J4.11 (Pin_11)
- new net opto_4_out: J4.12 (Pin_12)
- new net signal_ads: J17.7 (Pin_7)
- no-connect marks 0 -> 28
