File: electronics/data_acquisition.kicad_sch (KiCad schematic)
At the start: 0 parts

Commit message: version en dos placas, pero con errores de tierra general. Se procede a versionar la PCB
Parts:
- added C31, C32, C33, C34: C, symbol Device:C
- added J18: Screw_Terminal_01x01, symbol Connector:Screw_Terminal_01x01
- added R41, R42, R43, R44, R45, R46, R47, R48, R49: R, symbol Device:R
- added U10: OPA124U, Package_SO:SOIC-8_3.9x4.9mm_P1.27mm, symbol Amplifier_Operational:OPA121KU
- added U11: TL074, symbol Amplifier_Operational:TL074
Connections:
- new net: R44.1, U11.1, U11.2 (-)
- new net: R44.2, R45.1, R46.2, U11.6 (-)
- new net: C33.1, C34.1, U10.7 (V+)
- new net: R41.1, U10.2 (-)
- new net: R41.2, R42.1, U10.6
- new net: C31.1, C32.1, U10.4 (V-)
- new net: R47.2, R48.2, R49.1, U11.13 (-)
- new net: J18.1 (Pin_1), R49.2, U11.14
- new net: R47.1, U11.8, U11.9 (-)
- new net: R48.1, U11.11 (V-)
- new net: R46.1, U11.4 (V+)
- new net: R43.2, U10.3 (+)
- new net ADS_signal_out: R45.2, U11.7
- new net GND1: C31.2, C32.2, C33.2, C34.2, R43.1, U10.8 (Subst.), U11.12 (+), U11.5 (+)
- new net MCP_vbias_in: U11.10 (+)
- new net TIA_in: U11.3 (+)
- new net TIA_out: R42.2
- no-connect marks 0 -> 2
