File: electronics/piezo_control.kicad_sch (KiCad schematic)
At the start: 0 parts

Commit message: version en dos placas, pero con errores de tierra general. Se procede a versionar la PCB
Parts:
- added BZ1, BZ2, BZ3, BZ4: Buzzer, symbol Device:Buzzer
- added C15, C16, C17, C18, C19, C20, C21, C22, C23, C24, C25, C26, C27, C28, C29, C30, C35, C36, C37, C38, C39, C40, C41, C42, C43, C44, C45, C46: C, symbol Device:C
- added Q1, Q3, Q5, Q7: 2N3904, Package_TO_SOT_THT:TO-92_Inline, symbol Transistor_BJT:2N3904
- added Q2, Q4, Q6, Q8: 2N3906, Package_TO_SOT_THT:TO-92_Inline, symbol Transistor_BJT:2N3906
- added R10, R11, R12, R13, R14, R15, R16, R17, R18, R19, R20, R21, R22, R23, R24, R25, R26, R27, R28, R29, R30, R31, R32, R33, R34, R35, R36, R37, R38, R39, R40, R9: R, symbol Device:R
- added U3, U6, U7, U8, U9: TL074, symbol Amplifier_Operational:TL074
Connections:
- new net: C16.1, R10.2, U3.5 (+)
- new net: R15.1, U3.7
- new net: C37.2, C38.2, U6.4 (V+)
- new net: Q7.1 (E), Q8.1 (E), R40.1, U9.13 (-)
- new net: Q7.2 (B), Q8.2 (B), U9.14
- new net: C45.1, C46.1, U8.11 (V-)
- new net: C19.1, C21.1, U3.11 (V-)
- new net: Q3.1 (E), Q4.1 (E), R24.1, U9.6 (-)
- new net: Q3.2 (B), Q4.2 (B), U9.7
- new net: C22.1, R17.2, U6.3 (+)
- new net: R32.2, R33.1, U7.13 (-)
- new net: R33.2, U7.14, U9.10 (+)
- new net: C23.1, R18.2, U6.5 (+)
- new net: C17.1, R11.1, R14.2, R15.2, U3.9 (-)
- new net: C17.2, R11.2, R12.1, U3.8
- new net: C24.1, R19.2, R20.2, R21.1, U6.9 (-)
- new net: C24.2, R21.2, R22.1, U6.8
- new net: R22.2, R23.1, U6.13 (-)
- new net: C29.1, R29.2, R30.2, R31.1, U7.10 (+)
- new net: C29.2, R31.2, R32.1, U7.8
- new net: R12.2, R13.1, U3.13 (-)
- new net: R13.2, U3.14, U9.3 (+)
- new net: R38.2, R39.1, U8.13 (-)
- new net: R39.2, U8.14, U9.12 (+)
- new net: C27.1, R27.2, U8.3 (+)
- new net: C43.2, C44.2, U8.4 (V+)
- new net: C41.1, C42.1, U7.11 (V-)
- new net: BZ2.1 (+), R24.2
- new net: Q1.2 (B), Q2.2 (B), U9.1
- new net: Q1.1 (E), Q2.1 (E), R16.1, U9.2 (-)
- new net: BZ4.1 (+), R40.2
- new net: Q5.1 (E), Q6.1 (E), R34.1, U9.9 (-)
- new net: Q5.2 (B), Q6.2 (B), U9.8
- new net: R29.1, U7.1
- new net: C25.1, R25.2, U7.3 (+)
- new net: C26.1, R26.2, U7.5 (+)
- new net: R30.1, U7.7
- new net: C35.1, C36.1, U6.11 (V-)
- new net: R19.1, U6.1
- new net: R20.1, U6.7
- new net: C18.2, C20.2, U3.4 (V+)
- new net: C30.1, R35.2, R36.2, R37.1, U8.10 (+)
- new net: C30.2, R37.2, R38.1, U8.8
- new net: R35.1, U8.1
- new net: C28.1, R28.2, U8.5 (+)
- new net: R36.1, U8.7
- new net: R14.1, U3.1
- new net: C15.1, R9.2, U3.3 (+)
- new net: BZ1.1 (+), R16.2
- new net: C39.2, C40.2, U7.4 (V+)
- new net: R23.2, U6.14, U9.5 (+)
- new net: BZ3.1 (+), R34.2
- new net GNDA: BZ1.2 (-), BZ2.2 (-), BZ3.2 (-), BZ4.2 (-), C15.2, C16.2, C18.1, C19.2, C20.1, C21.2, C22.2, C23.2, C25.2, C26.2, C27.2, C28.2, C35.2, C36.2, C37.1, C38.1, C39.1, C40.1, C41.2, C42.2, C43.1, C44.1, C45.2, C46.2, U3.10 (+), U3.12 (+), U3.2 (-), U3.6 (-), U6.10 (+), U6.12 (+), U6.2 (-), U6.6 (-), U7.12 (+), U7.6 (-), U7.9 (-), U8.12 (+), U8.9 (-)
- new net MCP_coarse_r1_in: R10.1
- new net MCP_coarse_r2_in: R18.1
- new net MCP_coarse_r3_in: R26.1
- new net MCP_coarse_r4_in: R28.1
- new net MCP_fine_r1_in: R9.1
- new net MCP_fine_r2_in: R17.1
- new net MCP_fine_r3_in: R25.1
- new net MCP_fine_r4_in: R27.1
