File: electronics/power_supply.kicad_sch (KiCad schematic)
At the start: 43 parts, among them J1 17VAC_transformer, J2 sym_pow_17VDCsupply, J3 5VDC-3VDC_GND_out, U1 LM317, U2 LM337, U4 LM7805, U5 LM1117T-3.3

Commit message: version en dos placas, pero con errores de tierra general. Se procede a versionar la PCB
Parts:
- added C5: 100uF, Capacitor_THT:CP_Radial_D5.0mm_P2.00mm, symbol Device:C_Polarized
- added C7: 10uF, Capacitor_THT:CP_Radial_D5.0mm_P2.00mm, symbol Device:C_Polarized
- added H1, H2, H3, H4: MountingHole, MountingHole:MountingHole_3.2mm_M3, symbol Mechanical:MountingHole
- C11, C12: footprint Capacitor_THT:C_Radial_D5.0mm_H11.0mm_P2.00mm -> Capacitor_THT:CP_Radial_D5.0mm_P2.00mm
- C13: value 10uF -> 0.1uF; footprint Capacitor_THT:CP_Radial_D5.0mm_P2.00mm -> Capacitor_THT:C_Disc_D6.0mm_W2.5mm_P5.00mm
- C14: value 100uF -> 0.1uF; footprint Capacitor_THT:C_Disc_D5.0mm_W2.5mm_P2.50mm -> Capacitor_THT:C_Disc_D6.0mm_W2.5mm_P5.00mm
- C8: value 100nF -> 0.1uF
- D13: value Red_led -> Orange_led
- U5: footprint Package_TO_SOT_THT:TO-220-3_Horizontal_TabDown -> Package_TO_SOT_THT:TO-220-3_Vertical
- gave numbers to parts that had none: 1
Connections:
- net GND: now also C5.2, C7.2
- net +3.3V: now reaches C14.1, D12.2 (A), J3.2 (Pin_2), R8.1, U5.2 (VO)
- net +3.3V: now also C5.1
- net +5C: now reaches C13.1, C8.1, D11.2 (A), D12.1 (K), J3.1 (Pin_1), R7.1, U4.3 (VO), U5.3 (VI)
- net +5C: now also C7.1
- net +15V: now reaches C11.1, D2.2 (A), D4.1 (K), D6.1 (K), J2.1 (Pin_1), R1.1, R3.1, U1.2 (VO)
- net -15V: now reaches C12.2, D3.1 (K), D5.2 (A), D7.2 (A), D9.1 (K), J2.3 (Pin_3), R6.2, U2.3 (VO)
Other:
- company: Boo -> Boo Inventions
- title: Fuente_Low_Noise_STM -> Esquemático Fuente de Poder Bajo Ruido
- moved on the sheet: C1, C10, C11, C12, C13, C14, C2, C3, C4, C6, C8, C9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
