File: electronics/rough_approach.kicad_sch (KiCad schematic)
At the start: 0 parts

Commit message: version en dos placas, pero con errores de tierra general. Se procede a versionar la PCB
Parts:
- added J19: Conn_01x04_Socket, symbol Connector:Conn_01x04_Socket
- added J20: Conn_01x02_Socket, symbol Connector:Conn_01x02_Socket
- added R50, R51, R52, R53, R54, R55, R56, R57: R, symbol Device:R
- added U12, U13, U14, U15: PC817, Package_DIP:DIP-4_W7.62mm, symbol Isolator:PC817
Connections:
- new net: R52.1, U14.1
- new net: J19.3 (Pin_3), R56.1, U14.3
- new net: J20.1 (Pin_1), U12.4, U13.4, U14.4, U15.4
- new net: R51.1, U13.1
- new net: J19.2 (Pin_2), R55.1, U13.3
- new net: R50.1, U12.1
- new net: J19.1 (Pin_1), R54.1, U12.3
- new net: J19.4 (Pin_4), R57.1, U15.3
- new net: R53.1, U15.1
- new net DGND: U12.2, U13.2, U14.2, U15.2
- new net GNDPWR: J20.2 (Pin_2), R54.2, R55.2, R56.2, R57.2
- new net opto_1_in: R50.2
- new net opto_2_in: R51.2
- new net opto_3_in: R52.2
- new net opto_4_in: R53.2
